File: ch32ump/ch32ump.kicad_pcb (KiCad board)
At the start: 2 copper layers, 50.8 x 22.9 mm, 29 parts, among them J1 USB_B_Micro, J2 Conn_01x02, J3 Conn_01x16, J4 Conn_01x12, Q2 DMP2045U, SW1 SW_Push_Dual, U1 CH32V003F4P6, U2 AP2112K-3.3, U3 MCP73831-2-OT

Commit message: Saint Pipeline, please give me the green light
Parts:
- removed Q2: DMP2045U, Package_TO_SOT_SMD:SOT-23_Handsoldering
- removed R3: 100k, Resistor_SMD:R_0603_1608Metric_Pad0.98x0.95mm_HandSolder
- added C5: 1u, Capacitor_SMD:C_0402_1005Metric_Pad0.74x0.62mm_HandSolder, F.Cu at (14.7, 16.8)
- J2: footprint Connector_JST:JST_PH_S2B-PH-K_1x02_P2.00mm_Horizontal -> Connector_JST:JST_PH_S2B-PH-SM4-TB_1x02-1MP_P2.00mm_Horizontal
- R4: value 10k -> 100k
- moved D2 29.7 mm to (18.8, 4.70), turned to 180 degrees
- moved R1 23.4 mm to (44.5, 5.33)
- moved D1 20.2 mm to (28.0, 14.5)
- moved R6 19.3 mm to (18.4, 11.9), turned to 180 degrees
- moved C2 14.1 mm to (15.7, 6.22), turned to -90 degrees
- moved R8 13.9 mm to (28.0, 16.4), turned to 180 degrees
- moved R2 12.7 mm to (32.3, 5.44)
- moved R7 12.4 mm to (41.9, 5.33)
- moved C1 11.2 mm to (18.7, 7.11), turned to 180 degrees
- moved R5 11.0 mm to (18.4, 9.65), turned to 0 degrees
- moved NT1 7.95 mm to (30.0, 5.45), turned to 90 degrees
- moved U2 5.76 mm to (22.4, 8.06)
- moved U3 5.65 mm to (14.8, 10.9), turned to -90 degrees
- moved D3 5.40 mm to (10.7, 11.2), turned to 180 degrees
- moved C4 5.39 mm to (26.0, 7.11)
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Connections:
- C1 pad 1: Net-(D2-K) -> VBUS
- D2 pad 1: Net-(D2-K) -> VBUS
- D2 pad 2: VBUS -> +BATT
- J3 pad 3: unconnected-(J3-Pin_3-Pad3) -> AREF
- J4 pad 4: unconnected-(J4-Pin_4-Pad4) -> PC0
- R4 pad 2: Net-(D2-K) -> VBUS
- U2 pad 1: Net-(D2-K) -> VBUS
Routing:
- net D+: track 0.00 -> 82.3 mm, vias 0 -> 5
- net UTX: track 0.00 -> 46.4 mm, vias 0 -> 1
- net A3: track 0.00 -> 41.9 mm, vias 0 -> 2
- net D-: track 0.00 -> 41.2 mm, vias 0 -> 2
- net VBUS: track 0.00 -> 40.9 mm, vias 0 -> 1
- net PC0: track 0.00 -> 37.3 mm, vias 0 -> 1
- net ~{RESET}: track 0.00 -> 36.5 mm, vias 0 -> 2
- net URX: track 0.00 -> 27.7 mm, vias 0 -> 1
- net MI: track 0.00 -> 23.0 mm, vias 0 -> 1
- net PC4: track 0.00 -> 21.1 mm
- net MO: track 0.00 -> 21.0 mm, vias 0 -> 1
- net SCK: track 0.00 -> 21.0 mm, vias 0 -> 1
- net PA2: track 0.00 -> 20.9 mm
- net SCL: track 0.00 -> 20.5 mm
- net SDA: track 0.00 -> 19.7 mm
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- added copper zone on In2.Cu, net +3.3V
- added copper zone on In1.Cu, net GND
Other:
- copper layers 2 -> 4
