File: ch32ump/ch32ump.kicad_sch (KiCad schematic)
At the start: 25 parts, among them J1 USB_B_Micro, J2 Conn_01x02, J3 Conn_01x16, J4 Conn_01x12, Q2 DMP2045U, SW1 SW_Push_Dual, U1 CH32V003F4P6, U2 AP2112K-3.3, U3 MCP73831-2-OT

Commit message: Saint Pipeline, please give me the green light
Parts:
- removed Q2: DMP2045U, Package_TO_SOT_SMD:SOT-23_Handsoldering, symbol Device:Q_PMOS_Depletion
- removed R3: 100k, Resistor_SMD:R_0603_1608Metric_Pad0.98x0.95mm_HandSolder, symbol Device:R
- added C5: 1u, Capacitor_SMD:C_0402_1005Metric_Pad0.74x0.62mm_HandSolder, symbol Device:C
- J2: footprint Connector_JST:JST_PH_S2B-PH-K_1x02_P2.00mm_Horizontal -> Connector_JST:JST_PH_S2B-PH-SM4-TB_1x02-1MP_P2.00mm_Horizontal
- R4: value 10k -> 100k
Connections:
- net +BATT: now also D2.2 (A)
- net GND: now also C5.2
- net PC0: now also J4.4 (Pin_4)
- net VBUS: now also C1.1, D2.1 (K), R4.2, U2.1 (VIN); no longer D2.2 (A)
- net AREF: now reaches J3.3 (Pin_3)
- net AREF: now also C5.1
- no-connect marks 4 -> 3
Other:
- moved on the sheet: C2, D1, D2, J2, R1, R7, R8
